File: io-board/io-board.sch (KiCad schematic (older format))
At the start: 16 parts

Commit message: started working on the main-board
Connections:
- net labels added: PCINT19
- net labels removed: PCINT10
- wire segments 120 -> 121
Changed lines of the file:
@@
 LIBS:valves
 LIBS:74HCT595D_118
+LIBS:connector
 LIBS:ULN2004A
-LIBS:connector
-LIBS:kerbalkontrol-cache
 EELAYER 25 0
 EELAYER END
@@
 PCINT18
 Text GLabel 7200 2750 2    60   Input ~ 0
-PCINT10
+PCINT19
 Text GLabel 7200 2850 2    60   Input ~ 0
 PCINT20
@@
 P 9450 6150
 F 0 "#PWR?" H 9450 6000 50  0001 C CNN
-F 1 "+12V" H 9600 6300 0   0000 C CNN
+F 1 "+12V" H 9450 6300 60  0000 C CNN
 F 2 "" H 9450 6150 50  0000 C CNN
 F 3 "" H 9450 6150 50  0000 C CNN
@@
 P 9550 6150
 F 0 "#PWR?" H 9550 6000 50  0001 C CNN
-F 1 "+12V" H 9600 6300 50  0000 C CNN
+F 1 "+12V" H 9600 6300 0   0000 C CNN
 F 2 "" H 9550 6150 50  0000 C CNN
 F 3 "" H 9550 6150 50  0000 C CNN
@@
 P 9650 6150
 F 0 "#PWR?" H 9650 6000 50  0001 C CNN
-F 1 "+5V" H 9650 6290 0   0000 C CNN
+F 1 "+5V" H 9600 6300 60  0000 C CNN
 F 2 "" H 9650 6150 50  0000 C CNN
 F 3 "" H 9650 6150 50  0000 C CNN
@@
 P 9750 6150
 F 0 "#PWR?" H 9750 6000 50  0001 C CNN
-F 1 "+5V" H 9800 6300 50  0000 C CNN
+F 1 "+5V" H 9800 6300 0   0000 C CNN
 F 2 "" H 9750 6150 50  0000 C CNN
 F 3 "" H 9750 6150 50  0000 C CNN
@@
 P 9850 6150
 F 0 "#PWR?" H 9850 5900 50  0001 C CNN
-F 1 "GND" H 9900 6000 50  0000 C CNN
+F 1 "GND" H 9900 6000 0   0000 C CNN
 F 2 "" H 9850 6150 50  0000 C CNN
 F 3 "" H 9850 6150 50  0000 C CNN
@@
 P 9950 6150
 F 0 "#PWR?" H 9950 5900 50  0001 C CNN
-F 1 "GND" H 9950 6000 0   0000 C CNN
+F 1 "GND" H 9900 6000 60  0000 C CNN
 F 2 "" H 9950 6150 50  0000 C CNN
 F 3 "" H 9950 6150 50  0000 C CNN
@@
 Text GLabel 10050 6150 3    60   Input ~ 0
 SCL
+Wire Wire Line
+	9400 2400 9400 3900
 $EndSCHEMATC

Commit message: started routing io-board
Parts:
- C1, C2: renamed from C?; footprint (none) -> Capacitors_SMD:C_0603
- IC1, IC2: renamed from IC?; footprint (none) -> ULN2004A:SO16
- IC3: renamed from IC?; footprint TQFP32 -> Housings_QFP:TQFP-32_7x7mm_Pitch0.8mm
- J1: renamed from J?; footprint (none) -> Connect:RJ45_TRANSFO_ver2
- JP1: renamed from JP?; footprint (none) -> Pin_Headers:Pin_Header_Straight_1x03_Pitch2.54mm
- P1: renamed from P?; footprint (none) -> Pin_Headers:Pin_Header_Straight_2x16_Pitch2.54mm
- P2: renamed from P?; footprint (none) -> Pin_Headers:Pin_Header_Straight_2x08_Pitch2.54mm
- P3: renamed from P?; footprint (none) -> Pin_Headers:Pin_Header_Straight_2x14_Pitch2.54mm
- Y1: renamed from Y?; footprint (none) -> Crystals:Crystal_HC49-4H_Vertical
- gave numbers to parts that had none: 5
Other:
- moved on the sheet: P1
