File: io-board/io-board.sch (KiCad schematic (older format))
At the start: 16 parts, among them CON1 AVR-ISP-6, IC1 ULN2004A, IC2 ULN2004A, IC3 ATMEGA328P-A, J1 INTERFACE CONNECTOR, P1 SWITCHES, P2 INTERFACES, P3 LIGHTS, U1 74HCT595D,118, U2 74HCT595D,118, U3 74HCT595D,118, U4 74HCT595D,118, Y1 16Mhz

Commit message: fixed some routing
Parts:
- CON1: footprint AVR-ISP-6 -> Pin_Headers:Pin_Header_Straight_2x03_Pitch2.54mm
Changed lines of the file:
@@
 LIBS:contrib
 LIBS:valves
-LIBS:74HCT595D_118
-LIBS:connector
-LIBS:ULN2004A
 LIBS:io-board-cache
 EELAYER 25 0
@@
 F 0 "CON1" H 9745 2040 50  0000 C CNN
 F 1 "AVR-ISP-6" H 9585 1570 50  0000 L BNN
-F 2 "AVR-ISP-6" V 9330 1840 50  0001 C CNN
+F 2 "Pin_Headers:Pin_Header_Straight_2x03_Pitch2.54mm" V 9330 1840 50  0001 C CNN
 F 3 "" H 9825 1800 50  0000 C CNN
 	1    9850 1800

Commit message: started routing main-board
Parts:
- added R1: 10K, Resistors_SMD:R_0603, symbol R
Connections:
- wire segments 121 -> 122
Changed lines of the file:
@@
 LIBS:contrib
 LIBS:valves
+LIBS:74HCT595D_118
+LIBS:connector
+LIBS:ULN2004A
 LIBS:io-board-cache
 EELAYER 25 0
@@
 Text GLabel 10050 4100 0    60   Input ~ 0
 RX1
+Text GLabel 8250 1750 0    60   Input ~ 0
+RST
+$Comp
+L R R1
+U 1 1 591A9226
+P 8400 1600
+F 0 "R1" V 8480 1600 50  0000 C CNN
+F 1 "10K" V 8400 1600 50  0000 C CNN
+F 2 "Resistors_SMD:R_0603" V 8330 1600 50  0001 C CNN
+F 3 "" H 8400 1600 50  0000 C CNN
+	1    8400 1600
+	1    0    0    -1
+$EndComp
+Wire Wire Line
+	8250 1750 8400 1750
+$Comp
+L +5V #PWR034
+U 1 1 591A98CA
+P 8400 1450
+F 0 "#PWR034" H 8400 1300 50  0001 C CNN
+F 1 "+5V" H 8400 1590 50  0000 C CNN
+F 2 "" H 8400 1450 50  0000 C CNN
+F 3 "" H 8400 1450 50  0000 C CNN
+	1    8400 1450
+	1    0    0    -1
+$EndComp
 $EndSCHEMATC

Commit message: finished BOM
Parts:
- C1: value 22uF -> 22pf
- C2: value 22uF -> 22pF
- IC1, IC2: symbol ULN2004A -> ULN2004A-RESCUE-io-board
Changed lines of the file:
@@
 EESchema Schematic File Version 2
+LIBS:io-board-rescue
 LIBS:power
 LIBS:device
@@
 LIBS:contrib
 LIBS:valves
-LIBS:74HCT595D_118
-LIBS:connector
-LIBS:ULN2004A
 LIBS:io-board-cache
 EELAYER 25 0
@@
 P 10200 850
 F 0 "C1" H 10225 950 50  0000 L CNN
-F 1 "22uF" H 10225 750 50  0000 L CNN
+F 1 "22pf" H 10225 750 50  0000 L CNN
 F 2 "Capacitors_SMD:C_0603" H 10238 700 50  0001 C CNN
 F 3 "" H 10200 850 50  0000 C CNN
@@
 P 10200 1150
 F 0 "C2" H 10225 1250 50  0000 L CNN
-F 1 "22uF" H 10225 1050 50  0000 L CNN
+F 1 "22pF" H 10225 1050 50  0000 L CNN
 F 2 "Capacitors_SMD:C_0603" H 10238 1000 50  0001 C CNN
 F 3 "" H 10200 1150 50  0000 C CNN
@@
 SCL
 $Comp
-L ULN2004A IC1
+L ULN2004A-RESCUE-io-board IC1
 U 1 1 59195288
 P 3200 1150
@@
 MOSI
 $Comp
-L ULN2004A IC2
+L ULN2004A-RESCUE-io-board IC2
 U 1 1 59198CE3
 P 3200 2950
