File: io-board/_saved_io-board.sch (KiCad schematic (older format))
At the start: 16 parts, among them CON1 AVR-ISP-6, IC1 ULN2004A, IC2 ULN2004A, IC3 ATMEGA328P-A, J1 INTERFACE CONNECTOR, P1 SWITCHES, P2 INTERFACES, P3 LIGHTS, U1 74HCT595D,118, U2 74HCT595D,118, U3 74HCT595D,118, U4 74HCT595D,118, Y1 16Mhz

Commit message: finished routing io-board
Parts:
- J1: footprint Connect:RJ45_TRANSFO_ver2 -> w_conn_pc:rj45-wiznet-rb1-125bag1a
Changed lines of the file:
@@
 F 0 "J1" H 10000 6200 50  0000 C CNN
 F 1 "INTERFACE CONNECTOR" H 9650 6200 50  0000 C CNN
-F 2 "Connect:RJ45_TRANSFO_ver2" H 9800 5700 50  0001 C CNN
+F 2 "w_conn_pc:rj45-wiznet-rb1-125bag1a" H 9800 5700 50  0001 C CNN
 F 3 "" H 9800 5700 50  0000 C CNN
 	1    9800 5700
