File: io-board/io-board.kicad_pcb (KiCad board)
At the start: 2 copper layers, 50.8 x 67.3 mm, 15 parts, among them IC1 ULN2004A, IC2 ULN2004A, IC3 ATMEGA328P-A, J1 INTERFACE CONNECTOR, P1 SWITCHES, P2 INTERFACES, P3 LIGHTS, U1 74HCT595D,118, U2 74HCT595D,118, U3 74HCT595D,118, U4 74HCT595D,118, Y1 16Mhz

Commit message: finished routing io-board
Parts:
- J1: footprint Connect:RJ45_TRANSFO_ver2 -> w_conn_pc:rj45-wiznet-rb1-125bag1a
- moved J1 61.8 mm to (130.5, 68.2)
- moved C1 60.3 mm to (143.9, 71.5)
- moved C2 60.3 mm to (144.0, 85.2)
- moved IC1 60.3 mm to (134.5, 113.9)
- moved IC2 60.3 mm to (134.5, 94.9)
- moved IC3 60.3 mm to (156.1, 77.1)
- moved JP1 60.3 mm to (162.2, 66.7)
- moved P1 60.3 mm to (167.5, 121.5)
- moved P2 60.3 mm to (144.7, 63.1)
- moved P3 60.3 mm to (124.3, 121.5)
- moved U1 60.3 mm to (144.7, 113.9)
- moved U2 60.3 mm to (144.7, 94.9)
- moved U3 60.3 mm to (154.8, 113.9)
- moved U4 60.3 mm to (154.8, 94.9)
- moved Y1 60.3 mm to (143.9, 75.9)
Connections:
- P2 pad 1: Net-(P2-Pad1) -> RX1
Routing:
- net GND: track 71.1 -> 316.2 mm, vias 0 -> 5
- net +5V: track 0.00 -> 178.3 mm, vias 0 -> 13
- net /LIGHT_POWER: track 0.00 -> 113.4 mm, vias 0 -> 3
- net MOSI: track 0.00 -> 99.5 mm, vias 0 -> 7
- net SCK: track 27.0 -> 95.9 mm, vias 4 -> 7
- net +12V: track 0.00 -> 65.2 mm, vias 0 -> 1
- net /OE: track 27.0 -> 85.7 mm, vias 4 -> 8
- net SDA: track 0.00 -> 58.1 mm, vias 0 -> 2
- net SS: track 0.00 -> 49.1 mm, vias 0 -> 4
- net SCL: track 0.00 -> 48.7 mm, vias 0 -> 2
- net /RCLK: track 26.9 -> 70.9 mm, vias 4 -> 9
- net Net-(U2-Pad9): track 0.00 -> 41.9 mm, vias 0 -> 2
- net ADC0: track 0.00 -> 38.7 mm
- net ADC2: track 0.00 -> 29.6 mm
- net MISO: track 0.00 -> 29.1 mm, vias 0 -> 2
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- added copper zone on B.Cu, net GND
- added copper zone on F.Cu, net GND

Commit message: fixed some routing
Parts:
- added CON1: AVR-ISP-6, Pin_Headers:Pin_Header_Straight_2x03_Pitch2.54mm, F.Cu at (164.8, 73.7)
Routing:
- net RST: track 0.00 -> 39.3 mm, vias 0 -> 6
- net +5V: track 178.3 -> 195.9 mm
- net MISO: track 29.1 -> 45.9 mm, vias 2 -> 5
- net MOSI: track 99.5 -> 111.4 mm, vias 7 -> 9
- net SCK: track 95.9 -> 103.0 mm
- net +12V: track 65.2 -> 71.8 mm, vias 1 -> 3
- net GND: track 316.2 -> 313.0 mm

Commit message: started routing main-board
Parts:
- added R1: , Resistors_SMD:R_0603, F.Cu at (153.9, 67.7)
- ?: renamed from CON1; value AVR-ISP-6 -> (none)
- C1, C2: value 22uF -> (none)
- IC1, IC2: value ULN2004A -> (none)
- IC3: value ATMEGA328P-A -> (none)
- J1: value INTERFACE CONNECTOR -> INTERFACE
- JP1: value JUMPER3 -> (none)
- P1: value SWITCHES -> (none)
- P2: value INTERFACES -> (none)
- U1, U2, U3, U4: value 74HCT595D,118 -> (none)
- Y1: value 16Mhz -> (none)
Routing:
- net RST: track 39.3 -> 48.4 mm, vias 6 -> 8
- net +5V: track 195.9 -> 198.1 mm, vias 13 -> 14
Other:
- board text added: "GPIO"
- board text added: "HIGH POWER LIGHTS"
- board text added: "ICSP"
- board text added: "SWITCHES"

Commit message: Add branding
Parts:
- added G***: LOGO, custom:logomark.soldermask, B.Cu at (132.1, 115.6)
Other:
- board text added: "design by sudharshan"
