File: main-board/main-board.sch (KiCad schematic (older format))
At the start: 16 parts

Commit message: fixed some routing
Parts:
- added C? (x2): C, symbol C
- added C?: 100nF, symbol C
- added P?: CONN_01X02, symbol CONN_01X02
- added R?: 10K, symbol R
- added Y?: Crystal, symbol Crystal
- D? (x2): symbol LED -> LED-RESCUE-main-board
- P?: symbol USB_B -> USB_B-RESCUE-main-board
Connections:
- wire segments 28 -> 35
Other:
- moved on the sheet: C?, IC?, R?

Commit message: started routing main-board
Parts:
- added CON1: AVR-ISP-6, AVR-ISP-6, symbol AVR-ISP-6
- added J4: INTERFACE5, w_conn_pc:rj45-wiznet-rb1-125bag1a, symbol RJ45
- added J8: INTERFACE6, w_conn_pc:rj45-wiznet-rb1-125bag1a, symbol RJ45
- added R1, R2: R, Resistors_SMD:R_0603, symbol R
- C1, C2: renamed from C?; footprint (none) -> Capacitors_SMD:C_0603
- C3: renamed from C?; footprint (none) -> Capacitors_Tantalum_SMD:CP_Tantalum_Case-S_EIA-3216-12_Hand
- C4, C5, C6: renamed from C?; footprint (none) -> Capacitors_SMD:C_0603_HandSoldering
- D1, D2: renamed from D?; footprint (none) -> LEDs:LED_0603
- IC1: renamed from IC?; footprint TQFP32 -> Housings_QFP:TQFP-32_7x7mm_Pitch0.8mm
- IC2: renamed from IC?; footprint SSOP28-LD -> FT232RL:SSOP28-LD
- J1, J2, J3, J5, J6, J7: renamed from J?; footprint (none) -> w_conn_pc:rj45-wiznet-rb1-125bag1a
- P1: renamed from P?; footprint (none) -> Connect:USB_B
- P2: renamed from P?; footprint (none) -> Pin_Headers:Pin_Header_Straight_2x01_Pitch2.54mm
- R3, R4, R5: renamed from R?; footprint (none) -> Resistors_SMD:R_0603
- Y1: renamed from Y?; footprint (none) -> Crystals:Crystal_HC49-U_Vertical
Connections:
- net VCC is gone; now on net +5V: IC1.4 (VCC), IC1.6 (VCC)
- net +12V: now also J4.1, J4.2, J8.1, J8.2
- net +5V: now also CON1.2, J4.3, J4.4, J8.3, J8.4, R1.1, R2.1
- net GND: now also CON1.6, J4.5, J4.6, J8.5, J8.6
- net MISO: now also CON1.1
- net MOSI: now also CON1.4
- net RST: now also CON1.5
- net SCK: now also CON1.3
- net SCL: now also J4.7, J8.7, R1.2
- net SDA: now also J4.8, J8.8, R2.2
Other:
- moved on the sheet: C1, C2, C3, C4, C5, C6, D1, D2, IC2, P1, P2, R3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
