File: main-board/_saved_main-board.sch (KiCad schematic (older format))
At the start: 28 parts, among them CON1 AVR-ISP-6, IC1 ATMEGA328-A, IC2 FT232RL, J1 INTERFACE1, J2 INTERFACE3, J3 INTERFACE5, J4 INTERFACE5, J5 INTERFACE2, J6 INTERFACE4, J7 INTERFACE6, J8 INTERFACE6, P1 USB_B, P2 CONN_01X02, Y1 Crystal

Commit message: finished fixes for the board
Parts:
- CON1: footprint AVR-ISP-6 -> EdiCopter:PAD1X6
- P3: renamed from P?; footprint (none) -> Connectors_Molex:Molex_NanoFit_1x03x2.50mm_Straight
Changed lines of the file:
@@
 F 0 "CON1" H 7495 3940 50  0000 C CNN
 F 1 "AVR-ISP-6" H 7335 3470 50  0000 L BNN
-F 2 "AVR-ISP-6" V 7080 3740 50  0001 C CNN
+F 2 "EdiCopter:PAD1X6" V 7080 3740 50  0001 C CNN
 F 3 "" H 7575 3700 50  0000 C CNN
 	1    7600 3700
@@
 Connection ~ 5300 3250
 $Comp
-L CONN_01X03 P?
+L CONN_01X03 P3
 U 1 1 59242768
 P 7700 4350
-F 0 "P?" H 7700 4550 50  0000 C CNN
+F 0 "P3" H 7700 4550 50  0000 C CNN
 F 1 "power" V 7800 4350 50  0000 C CNN
-F 2 "" H 7700 4350 50  0000 C CNN
+F 2 "Connectors_Molex:Molex_NanoFit_1x03x2.50mm_Straight" H 7700 4350 50  0001 C CNN
 F 3 "" H 7700 4350 50  0000 C CNN
 	1    7700 4350
@@
 $EndComp
 $Comp
-L +12V #PWR?
+L +12V #PWR062
 U 1 1 59242CBD
 P 7500 4250
-F 0 "#PWR?" H 7500 4100 50  0001 C CNN
+F 0 "#PWR062" H 7500 4100 50  0001 C CNN
 F 1 "+12V" H 7450 4400 50  0000 C CNN
 F 2 "" H 7500 4250 50  0000 C CNN
@@
 $EndComp
 $Comp
-L +5V #PWR?
+L +5V #PWR063
 U 1 1 59242E6E
 P 7500 4450
-F 0 "#PWR?" H 7500 4300 50  0001 C CNN
+F 0 "#PWR063" H 7500 4300 50  0001 C CNN
 F 1 "+5V" H 7500 4590 60  0000 C CNN
 F 2 "" H 7500 4450 50  0000 C CNN
@@
 $EndComp
 $Comp
-L GND #PWR?
+L GND #PWR064
 U 1 1 59242F2B
 P 7500 4350
-F 0 "#PWR?" H 7500 4100 50  0001 C CNN
+F 0 "#PWR064" H 7500 4100 50  0001 C CNN
 F 1 "GND" H 7500 4200 60  0000 C CNN
 F 2 "" H 7500 4350 50  0000 C CNN
